Commit message: Updated the xacro

File: src/ros2_jazzy/urdf/oslsim.xacro (robot description, xacro)
@@ -1,4 +1,5 @@
 <?xml version="1.0"?>
 <robot name="oslsim" xmlns:xacro="http://www.ros.org/wiki/xacro">
+<xacro:property name="mesh_dir" value="$(find ros2_jazzy)"/>
   <!-- ========================= -->
   <!-- ROS 2 CONTROL INTERFACE  -->
@@ -37,5 +38,5 @@
     <plugin name="ros_gz_control" filename="libgz_ros2_control_system.so">
       <ros>
-        <param>file: file:///home/pika/Hari/leg/install/ros2_jazzy/share/ros2_jazzy/config/controllers.yaml</param>
+        <param>file: $(arg mesh_dir)/config/controllers.yaml</param>
       </ros>
     </plugin>
@@ -101,5 +102,5 @@
         rpy="0 0 0" />
       <geometry>
-        <mesh filename="file:///home/pika/Hari/leg/install/ros2_jazzy/share/ros2_jazzy/meshes/thigh.dae"/>
+        <mesh filename="$(arg mesh_dir)/meshes/thigh.dae"/>
       </geometry>
     </visual>
@@ -147,5 +148,5 @@
       <geometry>
         <mesh
-          filename="file:///home/pika/Hari/leg/install/ros2_jazzy/share/ros2_jazzy/meshes/socket.dae" />
+          filename="$(arg mesh_dir)/meshes/socket.dae" />
       </geometry>
       <material
@@ -180,5 +181,5 @@
     <limit effort="1.0" velocity="100" lower="-1.57" upper="1.57" />
   </joint>
-  <link name="robot_knee">
+  <!-- <link name="robot_knee">
     <inertial>
       <origin
@@ -201,5 +202,5 @@
       <geometry>
         <mesh
-          filename="file:///home/pika/Hari/leg/install/ros2_jazzy/share/ros2_jazzy/meshes/robot_knee.dae"
+          filename="$(arg mesh_dir)/meshes/robot_knee.dae"
           scale="0.001 0.001 0.001"/>
       </geometry>
@@ -218,5 +219,5 @@
       </geometry>
     </collision>
-  </link>
+  </link> -->
   <!-- ========================= -->
   <!-- SHIN + KNEE              -->
@@ -228,5 +229,5 @@
         rpy="0 0 0" />
       <geometry>
-        <mesh filename="file:///home/pika/Hari/leg/install/ros2_jazzy/share/ros2_jazzy/meshes/shin.dae"/>
+        <mesh filename="$(arg mesh_dir)/meshes/shin.dae"/>
       </geometry>
       <material
@@ -252,42 +253,4 @@
                ixy="-1.5e-05" ixz="-2.9e-06" iyz="1.27e-05"/>
     </inertial>
-  </link>
-  <link name="osl_shank">
-    <inertial>
-      <origin
-        xyz="0.00071137 -0.14671 0.059447"
-        rpy="0 0 0" />
-      <mass
-        value="0.1" />
-      <inertia
-        ixx="0.00092446"
-        ixy="-1.5017E-05"
-        ixz="2.9586E-06"
-        iyy="0.00064852"
-        iyz="-1.2701E-05"
-        izz="0.0013496" />
-    </inertial>
-    <visual>
-      <origin
-        xyz="0 0 0"
-        rpy="0 0 0" />
-      <geometry>
-        <mesh
-          filename="file:///home/pika/Hari/leg/install/ros2_jazzy/share/ros2_jazzy/meshes/osl_shank.dae" />
-      </geometry>
-      <material
-        name="">
-        <color
-          rgba="0.79216 0.81961 0.93333 1" />
-      </material>
-    </visual>
-    <collision>
-      <origin
-        xyz="0.00071137 -0.14671 0.059447"
-        rpy="0 0 0" />
-      <geometry>
-        <box size="0.1 0.35 0.1"/>
-      </geometry>
-    </collision>
   </link>
   <joint name="knee" type="revolute">
@@ -310,5 +273,5 @@
         rpy="0 0 0" />
       <geometry>
-        <mesh filename="file:///home/pika/Hari/leg/install/ros2_jazzy/share/ros2_jazzy/meshes/foot.dae"/>
+        <mesh filename="$(arg mesh_dir)/meshes/foot.dae"/>
       </geometry>
       <material
@@ -376,5 +339,5 @@
       <geometry>
         <mesh
-          filename="file:///home/pika/Hari/leg/install/ros2_jazzy/share/ros2_jazzy/meshes/osl_foot.dae" />
+          filename="$(arg mesh_dir)/meshes/osl_foot.dae" />
       </geometry>
       <material

Commit message: URDF completed for visualization

File: src/ros2_jazzy/urdf/oslsim.xacro (robot description, xacro)
@@ -1,9 +1,9 @@
 <?xml version="1.0"?>
 <robot name="oslsim" xmlns:xacro="http://www.ros.org/wiki/xacro">
-<xacro:property name="mesh_dir" value="$(find ros2_jazzy)"/>
+<xacro:property name="mesh_dir" value="package://ros2_jazzy"/>
   <!-- ========================= -->
   <!-- ROS 2 CONTROL INTERFACE  -->
   <!-- ========================= -->
-  <ros2_control name="OSLSimSystem" type="system">
+  <!-- <ros2_control name="OSLSimSystem" type="system">
     <hardware>
       <plugin>gazebo_ros2_control/GazeboSystem</plugin>
@@ -33,7 +33,7 @@
       <state_interface name="effort"/>
     </joint>
-  </ros2_control>
+  </ros2_control> -->
   <!-- Gazebo ROS 2 Control Plugin -->
-  <gazebo>
+  <!-- <gazebo>
     <plugin name="ros_gz_control" filename="libgz_ros2_control_system.so">
       <ros>
@@ -41,9 +41,10 @@
       </ros>
     </plugin>
-  </gazebo>
+  </gazebo> -->
   <!-- ========================= -->
   <!-- WORLD & BASE STRUCTURE   -->
   <!-- ========================= -->
-  <link name="world"/>
+  <link name="world">
+  </link>
   <link name="slider">
     <inertial>
@@ -77,20 +78,21 @@
       <parent link="slider"/>
       <child link="entity"/>
-      <origin xyz="0 0 -0.05" rpy="0 0 0"/>
-  </joint>
+      <origin xyz="0 0 -0.1" rpy="0 0 0"/>
+  </joint>
+  <link name="body">
+    <inertial>
+      <origin
+        xyz="0 0 0"
+        rpy="0 0 0" />
+      <mass value="0.1"/>
+      <inertia ixx="0.001" iyy="0.001" izz="0.001"
+               ixy="0" ixz="0" iyz="0"/>
+    </inertial>
+  </link>
   <joint name="root_joint" type="fixed">
     <parent link="entity"/>
     <child link="body"/>
-  </joint>
-  <link name="body">
-    <inertial>
-      <origin
-        xyz="0 0 0"
-        rpy="0 0 0" />
-      <mass value="0.1"/>
-      <inertia ixx="0.001" iyy="0.001" izz="0.001"
-               ixy="0" ixz="0" iyz="0"/>
-    </inertial>
-  </link>
+    <origin xyz="0 0 -0.1" rpy="0 0 0"/>
+  </joint>
   <!-- ========================= -->
   <!-- THIGH + HIP              -->
@@ -127,4 +129,12 @@
     </inertial>
   </link>
+  <joint name="hip" type="revolute">
+    <parent link="body"/>
+    <child link="thigh"/>
+    <origin xyz="0.0 0.0 0" rpy="0 0 0" />
+    <axis xyz="0 1 0" />
+    <limit effort="1.0" velocity="100" lower="-1.57" upper="1.57" />
+    <dynamics damping="0.5" friction="0.5"/>
+  </joint>
   <link name="socket">
     <inertial>
@@ -165,12 +175,4 @@
     </collision>
   </link>
-  <joint name="hip" type="revolute">
-    <parent link="body"/>
-    <child link="thigh"/>
-    <origin xyz="-0.03 -0.015 0" rpy="0 0 0" />
-    <axis xyz="-0.03 1 0" />
-    <limit effort="1.0" velocity="100" lower="-1.57" upper="1.57" />
-    <dynamics damping="0.5" friction="0.5"/>
-  </joint>
   <joint name="osl_hip" type="revolute">
     <parent link="body"/>
@@ -181,27 +183,27 @@
     <limit effort="1.0" velocity="100" lower="-1.57" upper="1.57" />
   </joint>
-  <!-- <link name="robot_knee">
-    <inertial>
-      <origin
-        xyz="0.0149 -0.105 -0.18907"
-        rpy="1.5708 0 0" />
+  <link name="osl_shin">
+    <inertial>
+      <origin
+        xyz="-0.097 -0.135 -0.018"
+        rpy="3.14 0.0 0" />
       <mass
         value="0.55993" />
       <inertia
-        ixx="0.045555"
-        ixy="-0.0028683"
-        ixz="-0.00027507"
-        iyy="0.018107"
-        iyz="0.0020012"
-        izz="0.04735" />
-    </inertial>
-    <visual>
-      <origin
-        xyz="0 0 0"
-        rpy="0 1 0" />
+        ixx="0.00092445"
+        ixy="-0.000015"
+        ixz="-0.00000296"
+        iyy="0.00064852"
+        iyz="0.0000127"
+        izz="0.0013496" />
+    </inertial>
+    <visual>
+      <origin
+        xyz="-0.097 0.065 0.03"
+        rpy="3.14 0.0 0" />
       <geometry>
         <mesh
-          filename="$(arg mesh_dir)/meshes/robot_knee.dae"
-          scale="0.001 0.001 0.001"/>
+          filename="$(arg mesh_dir)/meshes/osl_shin.STL"
+          scale="0.00091 0.00091 0.00091"/>
       </geometry>
       <material
@@ -213,11 +215,39 @@
     <collision>
       <origin
-        xyz="0.0149 -0.105 -0.18907"
-        rpy="1.5708 0 0" />
+        xyz="0 0.05 0.037"
+        rpy="3.14 0.0 0" />
       <geometry>
         <box size="0.15 0.3 0.15"/>
       </geometry>
     </collision>
-  </link> -->
+  </link>
+  <joint name="osl_knee" type="revolute">
+    <parent link="socket"/>
+    <child link="osl_shin"/>
+    <origin
+      xyz="0.0 -0.157865 -0.4427"
+      rpy="1.5708 0 0" />
+    <axis xyz="0 0 1"/>
+    <limit effort="1.0" velocity="100" lower="-1.57" upper="1.57" />
+    <dynamics damping="0.5" friction="0.5"/>
+  </joint>
+  <link name="osl_shin_imu">
+  </link>
+  <joint name="osl_shin_imu_joint" type="fixed">
+    <parent link="osl_shin"/>
+    <child link="osl_shin_imu"/>
+    <origin
+      xyz="0.0 -0.02 0.004"
+      rpy="1.57 0 0" />
+  </joint>
+  <link name="osl_ankle_imu">
+  </link>
+  <joint name="osl_ankle_imu_joint" type="fixed">
+    <parent link="osl_shin"/>
+    <child link="osl_ankle_imu"/>
+    <origin
+      xyz="0.00 -0.32 0.004"
+      rpy="1.57 0 0" />
+  </joint>
   <!-- ========================= -->
   <!-- SHIN + KNEE              -->
@@ -318,5 +348,15 @@
     </inertial>
   </link>
-  <!-- <link name="osl_foot">
+  <joint name="ankle" type="revolute">
+    <parent link="shin"/>
+    <child link="foot"/>
+    <origin
+      xyz="-0.00077967 -0.3134 -0.026811"
+      rpy="0 1.5708 0" />
+    <axis xyz="1 0 0"/>
+     <limit effort="1.0" velocity="100" lower="-1.57" upper="1.57" />
+    <dynamics damping="0.5" friction="0.5"/>
+  </joint>
+  <!-- <link name="osl_shank">
     <inertial>
       <origin
@@ -335,9 +375,10 @@
     <visual>
       <origin
-        xyz="0 0 0"
-        rpy="0.175 -1.5708 -3.1416" />
+        xyz="-0.068 -0.28 0.07"
+        rpy="-0.25 1.57 0" />
       <geometry>
         <mesh
-          filename="$(arg mesh_dir)/meshes/osl_foot.dae" />
+          filename="$(arg mesh_dir)/meshes/osl_shank.obj"
+          scale="0.0009 0.0009 0.0009"/>
       </geometry>
       <material
@@ -349,6 +390,6 @@
     <collision>
       <origin
-        xyz="0.03 -0.065 0.03"
-        rpy="0 -1.5708 0" />
+        xyz="-0.068 -0.28 0.07"
+        rpy="-0.25 1.57 0" />
       <geometry>
         <box size="0.0675 0.025 0.2"/>
@@ -375,29 +416,82 @@
       </surface>
     </collision>
-  </link> -->
-  <joint name="ankle" type="revolute">
-    <parent link="shin"/>
-    <child link="foot"/>
+  </link>
+  <joint name="osl_extension" type="fixed">
+    <parent link="osl_shin"/>
+    <child link="osl_shank"/>
+    <origin
+      xyz="0 -0.15 -0.04"
+      rpy="0 0 0" />
+  </joint> -->
+  <link name="osl_foot">
+     <inertial>
+      <origin
+        xyz="-0.006 -0.156 -0.025"
+        rpy="-0.25 0 0" />
+      <mass
+        value="0.01" />
+      <inertia
+        ixx="0.00051563"
+        ixy="-2.53E-06"
+        ixz="-1.60E-06"
+        iyy="0.00049449"
+        iyz="-0.000134"
+        izz="0.0001125" />
+    </inertial>
+    <visual>
+      <origin
+        xyz="-0.016 -0.101 -0.045"
+        rpy="-0.25 0 0" />
+      <geometry>
+        <mesh
+          filename="$(arg mesh_dir)/meshes/osl_foot.obj"
+          scale="0.00091 0.00091 0.00091"/>
+      </geometry>
+      <material
+        name="">
+        <color
+          rgba="0.0 0.80 0.0 1" />
+      </material>
+    </visual>
+    <collision>
+      <origin
+        xyz="-0.068 -0.28 0.07"
+        rpy="-0.25 1.57 0" />
+      <geometry>
+        <box size="0.0675 0.025 0.2"/>
+      </geometry>
+      <surface>
+        <friction>
+          <ode>
+            <mu>1.0</mu>
+            <mu2>1.0</mu2>
+            <fdir1>1 0 0</fdir1>
+            <slip1>0</slip1>
+            <slip2>0</slip2>
+          </ode>
+          <torsional>
+            <coefficient>0.0</coefficient>
+            <patch_radius>0</patch_radius>
+            <surface_radius>0</surface_radius>
+            <use_patch_radius>1</use_patch_radius>
+            <ode>
+              <slip>0</slip>
+            </ode>
+          </torsional>
+        </friction>
+      </surface>
+    </collision>
+  </link>
+  <joint name="osl_ankle" type="revolute">
+    <parent link="osl_shin"/>
+    <child link="osl_foot"/>
     <origin
       xyz="-0.00077967 -0.3134 -0.026811"
-      rpy="0 1.5708 0" />
+      rpy="0.21 1.5708 0" />
     <axis xyz="1 0 0"/>
      <limit effort="1.0" velocity="100" lower="-1.57" upper="1.57" />
     <dynamics damping="0.5" friction="0.5"/>
   </joint>
-  <link name="foot_heel">
-    <inertial>
-          <origin xyz="0 0 0" rpy="0 0 0"/>
-          <mass value="0.00001" />
-          <inertia ixx="1.6e-08" ixy="0.0" ixz="0.0" iyy="1.6e-08" iyz="0.0" izz="1.6e-08"/>
-      </inertial>
-      <collision>
-          <origin xyz="0 0 0" rpy="0 0 0"/>
-          <geometry>
-              <sphere radius="0.020"/>
-          </geometry>
-      </collision>
-  </link>
-  <!-- <link name="osl_foot_loadcell_link">
+  <!-- <link name="foot_heel">
     <inertial>
           <origin xyz="0 0 0" rpy="0 0 0"/>
@@ -412,9 +506,22 @@
       </collision>
   </link> -->
-  <joint name="foot_heel_joint" type="fixed">
+  <!-- <link name="osl_foot_loadcell_link">
+    <inertial>
+          <origin xyz="0 0 0" rpy="0 0 0"/>
+          <mass value="0.00001" />
+          <inertia ixx="1.6e-08" ixy="0.0" ixz="0.0" iyy="1.6e-08" iyz="0.0" izz="1.6e-08"/>
+      </inertial>
+      <collision>
+          <origin xyz="0 0 0" rpy="0 0 0"/>
+          <geometry>
+              <sphere radius="0.020"/>
+          </geometry>
+      </collision>
+  </link> -->
+  <!-- <joint name="foot_heel_joint" type="fixed">
       <parent link="foot"/>
       <child link="foot_heel"/>
       <origin xyz="0.03 -0.065 0" rpy="0 0 0"/>
-  </joint>
+  </joint> -->
   <!-- <joint name="osl_foot_loadcell_link_joint" type="fixed">
       <parent link="osl_foot"/>
@@ -425,5 +532,5 @@
   <!-- IMU SENSOR (ROS 2 OK)    -->
   <!-- ========================= -->
-  <gazebo reference="shin">
+  <!-- <gazebo reference="shin">
     <sensor name="shin_imu" type="imu">
       <topic>imu/osl_shank</topic>
@@ -444,4 +551,4 @@
       <update_rate>50</update_rate>
     </sensor>
-  </gazebo>
+  </gazebo> -->
 </robot>

Commit message: FIX: rendering in the gazebo

File: src/ros2_jazzy/urdf/oslsim.xacro (robot description, xacro)
@@ -2,44 +2,4 @@
 <robot name="oslsim" xmlns:xacro="http://www.ros.org/wiki/xacro">
 <xacro:property name="mesh_dir" value="package://ros2_jazzy"/>
-  <!-- ========================= -->
-  <!-- ROS 2 CONTROL INTERFACE  -->
-  <!-- ========================= -->
-  <!-- <ros2_control name="OSLSimSystem" type="system">
-    <hardware>
-      <plugin>gazebo_ros2_control/GazeboSystem</plugin>
-    </hardware>
-    <joint name="hip">
-      <command_interface name="effort"/>
-      <state_interface name="position"/>
-      <state_interface name="velocity"/>
-      <state_interface name="effort"/>
-    </joint>
-    <joint name="osl_hip">
-      <command_interface name="effort"/>
-      <state_interface name="position"/>
-      <state_interface name="velocity"/>
-      <state_interface name="effort"/>
-    </joint>
-    <joint name="knee">
-      <command_interface name="effort"/>
-      <state_interface name="position"/>
-      <state_interface name="velocity"/>
-      <state_interface name="effort"/>
-    </joint>
-    <joint name="ankle">
-      <command_interface name="effort"/>
-      <state_interface name="position"/>
-      <state_interface name="velocity"/>
-      <state_interface name="effort"/>
-    </joint>
-  </ros2_control> -->
-  <!-- Gazebo ROS 2 Control Plugin -->
-  <!-- <gazebo>
-    <plugin name="ros_gz_control" filename="libgz_ros2_control_system.so">
-      <ros>
-        <param>file: $(arg mesh_dir)/config/controllers.yaml</param>
-      </ros>
-    </plugin>
-  </gazebo> -->
   <!-- ========================= -->
   <!-- WORLD & BASE STRUCTURE   -->
@@ -61,8 +21,8 @@
   </link>
   <joint name="slider_joint" type="prismatic">
-      <origin xyz="0 0 0" rpy="0.0 0.0 0.0"/>
+      <origin xyz="0 0 1" rpy="0.0 0.0 0.0"/>
       <parent link="world" />
       <child link="slider" />
-      <axis xyz="1 0 0" />
+      <axis xyz="1 1 0" />
       <limit effort="1" lower="-10.0" upper="100.0" velocity="1" />
       <dynamics damping="0.05" friction="0.1"/>
@@ -160,9 +120,4 @@
           filename="$(arg mesh_dir)/meshes/socket.dae" />
       </geometry>
-      <material
-        name="">
-        <color
-          rgba="0.79216 0.81961 0.93333 1" />
-      </material>
     </visual>
     <collision>
@@ -170,4 +125,9 @@
         xyz="0.0149 -0.105 -0.18907"
         rpy="1.5708 0 0" />
+      <material
+        name="">
+        <color
+          rgba="0.79216 0.81961 0.93333 1" />
+      </material>
       <geometry>
         <box size="0.15 0.3 0.15"/>
@@ -207,8 +167,6 @@
           scale="0.00091 0.00091 0.00091"/>
       </geometry>
-      <material
-        name="">
-        <color
-          rgba="0.79216 0.81961 0.93333 1" />
+      <material name="blue_leg">
+        <color rgba="0.2 0.4 1.0 1"/>
       </material>
     </visual>
@@ -220,6 +178,18 @@
         <box size="0.15 0.3 0.15"/>
       </geometry>
-    </collision>
-  </link>
+      <material
+        name="">
+        <color
+          rgba="0.79216 0.81961 0.93333 1" />
+      </material>
+    </collision>
+  </link>
+  <gazebo reference="osl_shin">
+  <material>
+    <ambient>0.2 0.4 1 1</ambient>
+    <diffuse>0.2 0.4 1 1</diffuse>
+    <specular>0.1 0.1 0.1 1</specular>
+  </material>
+</gazebo>
   <joint name="osl_knee" type="revolute">
     <parent link="socket"/>
@@ -261,4 +231,12 @@
         <mesh filename="$(arg mesh_dir)/meshes/shin.dae"/>
       </geometry>
+    </visual>
+    <collision>
+      <origin
+        xyz="0.00071104 -0.14671 -0.059447"
+        rpy="0 0 0" />
+      <geometry>
+        <box size="0.1 0.35 0.1"/>
+      </geometry>
       <material
         name="">
@@ -266,12 +244,4 @@
           rgba="0.79216 0.81961 0.93333 1" />
       </material>
-    </visual>
-    <collision>
-      <origin
-        xyz="0.00071104 -0.14671 -0.059447"
-        rpy="0 0 0" />
-      <geometry>
-        <box size="0.1 0.35 0.1"/>
-      </geometry>
     </collision>
     <inertial>
@@ -305,4 +275,12 @@
         <mesh filename="$(arg mesh_dir)/meshes/foot.dae"/>
       </geometry>
+    </visual>
+    <collision>
+      <origin
+        xyz="0.029606 -0.065 0.05"
+        rpy="0 0 0" />
+      <geometry>
+        <box size="0.0675 0.025 0.2"/>
+      </geometry>
       <material
         name="">
@@ -310,12 +288,4 @@
           rgba="0.79216 0.81961 0.93333 1" />
       </material>
-    </visual>
-    <collision>
-      <origin
-        xyz="0.029606 -0.065 0.05"
-        rpy="0 0 0" />
-      <geometry>
-        <box size="0.0675 0.025 0.2"/>
-      </geometry>
       <surface>
         <friction>
@@ -448,9 +418,4 @@
           scale="0.00091 0.00091 0.00091"/>
       </geometry>
-      <material
-        name="">
-        <color
-          rgba="0.0 0.80 0.0 1" />
-      </material>
     </visual>
     <collision>
@@ -461,4 +426,9 @@
         <box size="0.0675 0.025 0.2"/>
       </geometry>
+      <material
+        name="">
+        <color
+          rgba="0.0 0.80 0.0 1" />
+      </material>
       <surface>
         <friction>
@@ -532,23 +502,89 @@
   <!-- IMU SENSOR (ROS 2 OK)    -->
   <!-- ========================= -->
-  <!-- <gazebo reference="shin">
-    <sensor name="shin_imu" type="imu">
-      <topic>imu/osl_shank</topic>
+  <gazebo reference="osl_ankle_imu">
+    <sensor name="ankle_imu" type="imu">
+      <always_on>true</always_on>
+      <update_rate>200</update_rate>
+      <visualize>true</visualize>
       <imu>
-        <frame>shin</frame>
+        <angular_velocity>
+          <x><noise type="gaussian"><mean>0</mean><stddev>0.0003</stddev></noise></x>
+          <y><noise type="gaussian"><mean>0</mean><stddev>0.0003</stddev></noise></y>
+          <z><noise type="gaussian"><mean>0</mean><stddev>0.0003</stddev></noise></z>
+        </angular_velocity>
+        <linear_acceleration>
+          <x><noise type="gaussian"><mean>0</mean><stddev>0.01</stddev></noise></x>
+          <y><noise type="gaussian"><mean>0</mean><stddev>0.01</stddev></noise></y>
+          <z><noise type="gaussian"><mean>0</mean><stddev>0.01</stddev></noise></z>
+        </linear_acceleration>
       </imu>
-      <always_on>true</always_on>
-      <update_rate>50</update_rate>
     </sensor>
   </gazebo>
-  <gazebo reference="foot">
-    <sensor name="foot_imu" type="imu">
-      <topic>imu/osl_foot</topic>
+  <gazebo reference="osl_shin_imu">
+    <sensor name="shin_imu" type="imu">
+      <always_on>true</always_on>
+      <update_rate>200</update_rate>
+      <visualize>true</visualize>
       <imu>
-        <frame>foot</frame>
+        <angular_velocity>
+          <x><noise type="gaussian"><mean>0</mean><stddev>0.0003</stddev></noise></x>
+          <y><noise type="gaussian"><mean>0</mean><stddev>0.0003</stddev></noise></y>
+          <z><noise type="gaussian"><mean>0</mean><stddev>0.0003</stddev></noise></z>
+        </angular_velocity>
+        <linear_acceleration>
+          <x><noise type="gaussian"><mean>0</mean><stddev>0.01</stddev></noise></x>
+          <y><noise type="gaussian"><mean>0</mean><stddev>0.01</stddev></noise></y>
+          <z><noise type="gaussian"><mean>0</mean><stddev>0.01</stddev></noise></z>
+        </linear_acceleration>
       </imu>
-      <always_on>true</always_on>
-      <update_rate>50</update_rate>
     </sensor>
-  </gazebo> -->
+  </gazebo>
+  <!-- ========================= -->
+  <!-- ROS 2 CONTROL INTERFACE  -->
+  <!-- ========================= -->
+  <ros2_control name="GazeboSystem" type="system">
+    <hardware>
+      <plugin>gz_ros2_control/GazeboSimSystem</plugin>
+    </hardware>
+    <joint name="slider_joint">
+      <command_interface name="position"/>
+      <state_interface name="position"/>
+      <state_interface name="velocity"/>
+    </joint>
+    <joint name="hip">
+      <command_interface name="position" />
+      <state_interface name="position" />
+      <state_interface name="velocity"/>
+    </joint>
+    <joint name="osl_hip">
+      <command_interface name="position" />
+      <state_interface name="position" />
+      <state_interface name="velocity"/>
+    </joint>
+    <joint name="knee">
+      <command_interface name="position" />
+      <state_interface name="position" />
+      <state_interface name="velocity"/>
+    </joint>
+    <joint name="osl_knee">
+      <command_interface name="position" />
+      <state_interface name="position" />
+      <state_interface name="velocity"/>
+    </joint>
+    <joint name="ankle">
+      <command_interface name="position" />
+      <state_interface name="position" />
+      <state_interface name="velocity"/>
+    </joint>
+    <joint name="osl_ankle">
+      <command_interface name="position" />
+      <state_interface name="position" />
+      <state_interface name="velocity"/>
+    </joint>
+  </ros2_control>
+  <gazebo>
+    <plugin filename="gz_ros2_control-system" name="gz_ros2_control::GazeboSimROS2ControlPlugin">
+      <parameters>$(find ros2_jazzy)/config/controllers.yaml</parameters>
+    </plugin>
+  </gazebo>
 </robot>
