Commit message: FIX: not working on other pc due to directory conflicts

File: src/ros2_jazzy/urdf/newoslsim.xacro (robot description, xacro)
@@ -516,9 +516,9 @@
   <gazebo reference="osl_foot_loadcell_link">
     <sensor name='sensor_contact' type='contact'>
-      <always_on>true</always_on>
-      <update_rate>50</update_rate>
-      <topic>contact/foot</topic>
+      <!-- <always_on>true</always_on> -->
+      <!-- <update_rate>50</update_rate> -->
+      <!-- <topic>contact/foot</topic> -->
       <contact>
-          <collision>osl_foot_loadcell_link_collision_1</collision>
+          <collision>osl_foot_loadcell_link_collision_1_collision_1</collision>
       </contact>
     </sensor>
@@ -595,4 +595,13 @@
   </gazebo>
   <gazebo>
+    <plugin filename="gz-sim-touchplugin-system"
+          name="gz::sim::systems::TouchPlugin">
+      <target>ground_plane</target>
+      <namespace>foot</namespace>
+      <time>0.001</time>
+      <enabled>true</enabled>
+    </plugin>
+  </gazebo>
+  <gazebo>
     <plugin filename="gz-sim-contact-system"
         name="gz::sim::systems::Contact">

Commit message: UPDATE: fix the urdf with world

File: src/ros2_jazzy/urdf/newoslsim.xacro (robot description, xacro)
@@ -2,26 +2,26 @@
 <robot name="oslsim" xmlns:xacro="http://www.ros.org/wiki/xacro">
     <xacro:property name="mesh_dir" value="package://ros2_jazzy"/>
-    <link name="base_link">
-      <inertial>
+  <link name="world"/>
+  <link name="base_link">
+    <inertial>
+      <origin rpy="0.0 0 0" xyz="0 0 0"/>
+      <mass value="0.00001" />
+      <inertia ixx="1.0e-07" ixy="0.0" ixz="0.0" iyy="1.0e-07" iyz="0.0" izz="1.0e-07"/>
+    </inertial>
+  </link>
+  <joint name="base_link_joint" type="fixed">
+    <parent link="world" />
+      <child link="base_link" />
+  </joint>
+  <link name="slider">
+    <!-- <visual>
+    </visual> -->
+    <inertial>
         <origin rpy="0.0 0 0" xyz="0 0 0"/>
         <mass value="0.001" />
         <inertia ixx="1.0e-07" ixy="0.0" ixz="0.0" iyy="1.0e-07" iyz="0.0" izz="1.0e-07"/>
     </inertial>
-    </link>
-  <link name="slider">
-    <!-- <visual>
-    </visual> -->
-    <inertial>
-        <origin rpy="0.0 0 0" xyz="0 0 0"/>
-        <mass value="0.001" />
-        <inertia ixx="1.0e-07" ixy="0.0" ixz="0.0" iyy="1.0e-07" iyz="0.0" izz="1.0e-07"/>
-    </inertial>
     <collision>
         <origin rpy="0.0 0 0" xyz="0 0 0"/>
-        <material>
-          <ambient>1 0 0 1</ambient>
-          <diffuse>1 0 0 1</diffuse>
-          <specular>0.1 0.1 0.1 1</specular>
-        </material>
         <geometry>
             <box size="0.25 0.25 0.01"/>
@@ -29,4 +29,11 @@
     </collision>
   </link>
+  <gazebo reference="slider">
+      <kp>1000.0</kp>
+      <kd>1000.0</kd>
+      <mu1>0.5</mu1>
+      <mu2>0.5</mu2>
+      <material>Gazebo/Red</material>
+  </gazebo>
   <joint name="slider_joint" type="prismatic">
       <origin xyz="0 0 0" rpy="0.0 0.0 0.0"/>
@@ -44,4 +51,11 @@
         </inertial>
   </link>
+  <gazebo reference="entity">
+      <kp>1000.0</kp>
+      <kd>1000.0</kd>
+      <mu1>0.5</mu1>
+      <mu2>0.5</mu2>
+      <material>Gazebo/Blue</material>
+  </gazebo>
   <joint name="entity_joint" type="fixed">
       <parent link="slider"/>
@@ -65,4 +79,10 @@
     </inertial>
   </link>
+  <gazebo reference="body">
+      <kp>1000.0</kp>
+      <kd>1000.0</kd>
+      <mu1>0.5</mu1>
+      <mu2>0.5</mu2>
+  </gazebo>
   <joint name="root_joint" type="fixed">
     <parent link="entity"/>
@@ -107,27 +127,12 @@
         <box size="0.15 0.3 0.15"/>
       </geometry>
-      <!-- <material
-        name="">
-        <color
-          rgba="0.79216 0.81961 0.93333 1" />
-      </material> -->
-      <surface>
-          <friction>
-            <ode>
-              <mu>0.5</mu>
-              <mu2>0.5</mu2>
-            </ode>
-          </friction>
-          <contact>
-            <ode>
-              <kp>1000.0</kp>
-              <kd>1000.0</kd>
-              <max_vel>0.01</max_vel>
-              <min_depth>0.001</min_depth>
-            </ode>
-          </contact>
-        </surface>
     </collision>
   </link>
+  <gazebo reference="thigh">
+      <kp>1000.0</kp>
+      <kd>1000.0</kd>
+      <mu1>0.5</mu1>
+      <mu2>0.5</mu2>
+  </gazebo>
   <joint name="hip" type="revolute">
     <parent link="body"/>
@@ -178,4 +183,10 @@
     </collision>
   </link>
+  <gazebo reference="socket">
+      <kp>1000.0</kp>
+      <kd>1000.0</kd>
+      <mu1>0.5</mu1>
+      <mu2>0.5</mu2>
+  </gazebo>
   <joint name="osl_hip" type="revolute">
     <parent link="body"/>
@@ -226,4 +237,10 @@
     </collision>
   </link>
+  <gazebo reference="shin">
+      <kp>1000.0</kp>
+      <kd>1000.0</kd>
+      <mu1>0.5</mu1>
+      <mu2>0.5</mu2>
+  </gazebo>
   <joint name="knee"
     type="revolute">
@@ -281,4 +298,8 @@
   </link>
   <gazebo reference="osl_shank">
+    <kp>1000.0</kp>
+    <kd>1000.0</kd>
+    <mu1>0.5</mu1>
+    <mu2>0.5</mu2>
     <!-- Native gz-sim IMU sensor -->
     <sensor name="osl_foot_imu" type="imu">
@@ -369,4 +390,10 @@
     </collision>
   </link>
+  <gazebo reference="foot">
+      <kp>1000.0</kp>
+      <kd>1000.0</kd>
+      <mu1>1.0</mu1>
+      <mu2>1.0</mu2>
+  </gazebo>
   <joint name="ankle"
     type="revolute">
@@ -475,4 +502,10 @@
       </collision>
   </link>
+  <gazebo reference="foot_heel">
+      <kp>1000.0</kp>
+      <kd>1000.0</kd>
+      <mu1>0.5</mu1>
+      <mu2>0.5</mu2>
+  </gazebo>
   <joint name="foot_heel_joint" type="fixed">
       <parent link="foot"/>
@@ -491,22 +524,12 @@
               <sphere radius="0.020"/>
           </geometry>
-          <surface>
-            <friction>
-              <ode>
-                <mu>0.5</mu>
-                <mu2>0.5</mu2>
-              </ode>
-            </friction>
-            <contact>
-              <ode>
-                <kp>1000.0</kp>
-                <kd>1000.0</kd>
-                <max_vel>0.01</max_vel>
-                <min_depth>0.001</min_depth>
-              </ode>
-            </contact>
-          </surface>
       </collision>
   </link>
+  <gazebo reference="osl_foot_loadcell_link">
+      <kp>1000.0</kp>
+      <kd>1000.0</kd>
+      <mu1>0.5</mu1>
+      <mu2>0.5</mu2>
+  </gazebo>
   <joint name="osl_foot_loadcell_link_joint" type="fixed">
       <parent link="osl_foot"/>
@@ -608,5 +631,5 @@
       filename="gz-sim-odometry-publisher-system"
       name="gz::sim::systems::OdometryPublisher">
-      <odom_frame>odom</odom_frame>
+      <odom_frame>world</odom_frame>
       <robot_base_frame>base_link</robot_base_frame>
       <odom_topic>oslsim/odom</odom_topic>

Commit message: Fix : Changes to restore previous version

File: src/ros2_jazzy/urdf/newoslsim.xacro (robot description, xacro)
@@ -1,10 +1,11 @@
-<robot xmlns:ns0="http://www.ros.org/wiki/xacro" name="oslsim">
-    <ns0:arg name="mesh_dir" default="package://ros2_jazzy" />
-  <link name="world" />
+<?xml version="1.0"?>
+<robot name="oslsim" xmlns:xacro="http://www.ros.org/wiki/xacro">
+    <xacro:property name="mesh_dir" value="package://ros2_jazzy"/>
+  <link name="world"/>
   <link name="base_link">
     <inertial>
-      <origin rpy="0.0 0 0" xyz="0 0 0" />
+      <origin rpy="0.0 0 0" xyz="0 0 0"/>
       <mass value="0.00001" />
-      <inertia ixx="1.0e-07" ixy="0.0" ixz="0.0" iyy="1.0e-07" iyz="0.0" izz="1.0e-07" />
+      <inertia ixx="1.0e-07" ixy="0.0" ixz="0.0" iyy="1.0e-07" iyz="0.0" izz="1.0e-07"/>
     </inertial>
   </link>
@@ -12,16 +13,17 @@
     <parent link="world" />
       <child link="base_link" />
-      <origin xyz="0 0 0.15" rpy="0 0 0" />
   </joint>
   <link name="slider">
-    <inertial>
-        <origin rpy="0.0 0 0" xyz="0 0 0" />
+    <!-- <visual>
+    </visual> -->
+    <inertial>
+        <origin rpy="0.0 0 0" xyz="0 0 0"/>
         <mass value="0.001" />
-        <inertia ixx="1.0e-07" ixy="0.0" ixz="0.0" iyy="1.0e-07" iyz="0.0" izz="1.0e-07" />
+        <inertia ixx="1.0e-07" ixy="0.0" ixz="0.0" iyy="1.0e-07" iyz="0.0" izz="1.0e-07"/>
     </inertial>
     <collision>
-        <origin rpy="0.0 0 0" xyz="0 0 0" />
+        <origin rpy="0.0 0 0" xyz="0 0 0"/>
         <geometry>
-            <box size="0.25 0.25 0.01" />
+            <box size="0.25 0.25 0.01"/>
         </geometry>
     </collision>
@@ -35,16 +37,16 @@
   </gazebo>
   <joint name="slider_joint" type="prismatic">
-      <origin xyz="0 0 0" rpy="0.0 0.0 0.0" />
+      <origin xyz="0 0 0" rpy="0.0 0.0 0.0"/>
       <parent link="base_link" />
       <child link="slider" />
       <axis xyz="1 0 0" />
       <limit effort="1" lower="-10.0" upper="100.0" velocity="1" />
-      <dynamics damping="0.05" friction="0.1" />
+      <dynamics damping="0.05" friction="0.1"/>
   </joint>
   <link name="entity">
       <inertial>
-            <origin rpy="0.0 0 0" xyz="0 0 0" />
+            <origin rpy="0.0 0 0" xyz="0 0 0"/>
             <mass value="0.1" />
-            <inertia ixx="4.16666666667e-05" ixy="0.0" ixz="0.0" iyy="4.16666666667e-05" iyz="0.0" izz="4.16666666667e-05" />
+            <inertia ixx="4.16666666667e-05" ixy="0.0" ixz="0.0" iyy="4.16666666667e-05" iyz="0.0" izz="4.16666666667e-05"/>
         </inertial>
   </link>
@@ -57,13 +59,22 @@
   </gazebo>
   <joint name="entity_joint" type="fixed">
-      <parent link="slider" />
-      <child link="entity" />
-      <origin xyz="0 0 -0.05" rpy="0 0 0" />
+      <parent link="slider"/>
+      <child link="entity"/>
+      <origin xyz="0 0 -0.05" rpy="0 0 0"/>
   </joint>
   <link name="body">
     <inertial>
-      <origin xyz="0 0 0" rpy="0 0 0" />
-      <mass value="0.1" />
-      <inertia ixx="0.001" ixy="0" ixz="0" iyy="0.001" iyz="0" izz="0.001" />
+      <origin
+        xyz="0 0 0"
+        rpy="0 0 0" />
+      <mass
+        value="0.1" />
+      <inertia
+        ixx="0.001"
+        ixy="0"
+        ixz="0"
+        iyy="0.001"
+        iyz="0"
+        izz="0.001" />
     </inertial>
   </link>
@@ -75,17 +86,29 @@
   </gazebo>
   <joint name="root_joint" type="fixed">
-    <parent link="entity" />
-    <child link="body" />
+    <parent link="entity"/>
+    <child link="body"/>
   </joint>
   <link name="thigh">
     <inertial>
-      <origin xyz="0.0079 0.105 -0.18514" rpy="1.5708 0 0" />
-      <mass value="5.0" />
-      <inertia ixx="0.0451" ixy="-0.0023863" ixz="0.00041503" iyy="0.017843" iyz="-0.00079008" izz="0.046937" />
+      <origin
+        xyz="0.0079 0.105 -0.18514"
+        rpy="1.5708 0 0" />
+      <mass
+        value="0.55797" />
+      <inertia
+        ixx="0.0451"
+        ixy="-0.0023863"
+        ixz="0.00041503"
+        iyy="0.017843"
+        iyz="-0.00079008"
+        izz="0.046937" />
     </inertial>
     <visual>
-      <origin xyz="0 0 -0.004" rpy="0 0 0" />
-      <geometry>
-        <mesh filename="$(arg mesh_dir)/meshes/thigh.dae" />
+      <origin
+        xyz="0 0 -0.004"
+        rpy="0 0 0" />
+      <geometry>
+        <mesh
+          filename="$(arg mesh_dir)/meshes/thigh.dae" />
       </geometry>
       <material name="">
@@ -98,7 +121,9 @@
     </visual>
     <collision>
-      <origin xyz="0.0079 0.105 -0.18514" rpy="1.5708 0 0" />
-      <geometry>
-        <box size="0.01 0.01 0.01" />
+      <origin
+        xyz="0.0079 0.105 -0.18514"
+        rpy="1.5708 0 0" />
+      <geometry>
+        <box size="0.15 0.3 0.15"/>
       </geometry>
     </collision>
@@ -111,21 +136,33 @@
   </gazebo>
   <joint name="hip" type="revolute">
-    <parent link="body" />
-    <child link="thigh" />
+    <parent link="body"/>
+    <child link="thigh"/>
     <origin xyz="-0.03 -0.015 0" rpy="0 0 0" />
     <axis xyz="-0.03 1 0" />
-    <dynamics damping="0.5" friction="0.5" />
+    <dynamics damping="0.5" friction="0.5"/>
     <limit effort="1.0" velocity="100" lower="-1.57" upper="1.57" />
   </joint>
     <link name="socket">
     <inertial>
-      <origin xyz="0.0149 -0.105 -0.18907" rpy="1.5708 0 0" />
-      <mass value="5.0" />
-      <inertia ixx="0.045555" ixy="-0.0028683" ixz="-0.00027507" iyy="0.018107" iyz="0.0020012" izz="0.04735" />
+      <origin
+        xyz="0.0149 -0.105 -0.18907"
+        rpy="1.5708 0 0" />
+      <mass
+        value="0.55993" />
+      <inertia
+        ixx="0.045555"
+        ixy="-0.0028683"
+        ixz="-0.00027507"
+        iyy="0.018107"
+        iyz="0.0020012"
+        izz="0.04735" />
     </inertial>
     <visual>
-      <origin xyz="0 0 0" rpy="0 0 0" />
-      <geometry>
-        <mesh filename="$(arg mesh_dir)/meshes/socket.dae" />
+      <origin
+        xyz="0 0 0"
+        rpy="0 0 0" />
+      <geometry>
+        <mesh
+          filename="$(arg mesh_dir)/meshes/socket.dae" />
       </geometry>
       <material name="">
@@ -138,7 +175,9 @@
     </visual>
     <collision>
-      <origin xyz="0.0149 -0.105 -0.18907" rpy="1.5708 0 0" />
-      <geometry>
-        <box size="0.01 0.01 0.01" />
+      <origin
+        xyz="0.0149 -0.105 -0.18907"
+        rpy="1.5708 0 0" />
+      <geometry>
+        <box size="0.15 0.3 0.15"/>
       </geometry>
     </collision>
@@ -151,21 +190,33 @@
   </gazebo>
   <joint name="osl_hip" type="revolute">
-    <parent link="body" />
-    <child link="socket" />
+    <parent link="body"/>
+    <child link="socket"/>
     <origin xyz="0 0.015 0" rpy="0 0 0" />
     <axis xyz="0 1 0" />
-    <dynamics damping="0.5" friction="0.5" />
+    <dynamics damping="0.5" friction="0.5"/>
     <limit effort="1.0" velocity="100" lower="-1.57" upper="1.57" />
   </joint>
   <link name="shin">
     <inertial>
-      <origin xyz="0.00071104 -0.14671 -0.059447" rpy="0 0 0" />
-      <mass value="3.0" />
-      <inertia ixx="0.00092445" ixy="-1.5017E-05" ixz="-2.9597E-06" iyy="0.00064852" iyz="1.2705E-05" izz="0.0013496" />
+      <origin
+        xyz="0.00071104 -0.14671 -0.059447"
+        rpy="0 0 0" />
+      <mass
+        value="0.1" />
+      <inertia
+        ixx="0.00092445"
+        ixy="-1.5017E-05"
+        ixz="-2.9597E-06"
+        iyy="0.00064852"
+        iyz="1.2705E-05"
+        izz="0.0013496" />
     </inertial>
     <visual>
-      <origin xyz="0.006 0.01 0.006" rpy="0 0 0" />
-      <geometry>
-        <mesh filename="$(arg mesh_dir)/meshes/shin.dae" />
+      <origin
+        xyz="0.006 0.01 0.006"
+        rpy="0 0 0" />
+      <geometry>
+        <mesh
+          filename="$(arg mesh_dir)/meshes/shin.dae" />
       </geometry>
       <material name="">
@@ -178,7 +229,9 @@
     </visual>
     <collision>
-      <origin xyz="0.00071104 -0.14671 -0.059447" rpy="0 0 0" />
-      <geometry>
-        <box size="0.01 0.01 0.01" />
+      <origin
+        xyz="0.00071104 -0.14671 -0.059447"
+        rpy="0 0 0" />
+      <geometry>
+        <box size="0.1 0.35 0.1"/>
       </geometry>
     </collision>
@@ -190,22 +243,40 @@
       <mu2>0.5</mu2>
   </gazebo>
-  <joint name="knee" type="revolute">
-    <origin xyz="-0.0073766 0.057865 -0.4427" rpy="1.5708 0 0" />
-    <parent link="thigh" />
-    <child link="shin" />
-    <axis xyz="0 0 1" />
-    <dynamics damping="0.5" friction="0.5" />
+  <joint name="knee"
+    type="revolute">
+    <origin
+      xyz="-0.0073766 0.057865 -0.4427"
+      rpy="1.5708 0 0" />
+    <parent
+      link="thigh" />
+    <child
+      link="shin" />
+    <axis
+      xyz="0 0 1" />
+    <dynamics damping="0.5" friction="0.5"/>
     <limit effort="1.0" velocity="100" lower="-1.57" upper="1.57" />
   </joint>
   <link name="osl_shank">
     <inertial>
-      <origin xyz="0.00071137 -0.14671 0.059447" rpy="0 0 0" />
-      <mass value="3.0" />
-      <inertia ixx="0.00092446" ixy="-1.5017E-05" ixz="2.9586E-06" iyy="0.00064852" iyz="-1.2701E-05" izz="0.0013496" />
+      <origin
+        xyz="0.00071137 -0.14671 0.059447"
+        rpy="0 0 0" />
+      <mass
+        value="0.1" />
+      <inertia
+        ixx="0.00092446"
+        ixy="-1.5017E-05"
+        ixz="2.9586E-06"
+        iyy="0.00064852"
+        iyz="-1.2701E-05"
+        izz="0.0013496" />
     </inertial>
     <visual>
-      <origin xyz="0 0 0" rpy="0 0 0" />
-      <geometry>
-        <mesh filename="$(arg mesh_dir)/meshes/osl_shank.dae" />
+      <origin
+        xyz="0 0 0"
+        rpy="0 0 0" />
+      <geometry>
+        <mesh
+          filename="$(arg mesh_dir)/meshes/osl_shank.dae" />
       </geometry>
       <material name="">
@@ -218,7 +289,9 @@
     </visual>
     <collision>
-      <origin xyz="0.00071137 -0.14671 0.059447" rpy="0 0 0" />
-      <geometry>
-        <box size="0.01 0.01 0.01" />
+      <origin
+        xyz="0.00071137 -0.14671 0.059447"
+        rpy="0 0 0" />
+      <geometry>
+        <box size="0.1 0.35 0.1"/>
       </geometry>
     </collision>
@@ -229,30 +302,49 @@
     <mu1>0.5</mu1>
     <mu2>0.5</mu2>
-    <sensor name="osl_shank_imu" type="imu">
+    <!-- Native gz-sim IMU sensor -->
+    <sensor name="osl_foot_imu" type="imu">
       <always_on>true</always_on>
       <update_rate>50</update_rate>
       <visualize>true</visualize>
-      <topic>/imu/osl_shank</topic>
+      <topic>imu/osl_shank</topic>
       <pose>0 0 0 0 0 0</pose>
     </sensor>
     </gazebo>
-<joint name="osl_knee" type="revolute">
-    <origin xyz="-0.0073766 -0.062441 -0.4427" rpy="1.5708 0 0" />
-    <parent link="socket" />
-    <child link="osl_shank" />
-    <axis xyz="0 0 1" />
-    <dynamics damping="0.5" friction="0.5" />
-    <limit effort="200.0" velocity="100" lower="-1.57" upper="1.57" />
+<joint name="osl_knee"
+    type="revolute">
+    <origin
+      xyz="-0.0073766 -0.062441 -0.4427"
+      rpy="1.5708 0 0" />
+    <parent
+      link="socket" />
+    <child
+      link="osl_shank" />
+    <axis
+      xyz="0 0 1" />
+    <dynamics damping="0.5" friction="0.5"/>
+    <limit effort="1.0" velocity="100" lower="-1.57" upper="1.57" />
   </joint>
   <link name="foot">
     <inertial>
-      <origin xyz="0.029606 -0.056108 0.013102" rpy="-0.175 0 0" />
-      <mass value="1.0" />
-      <inertia ixx="0.00051563" ixy="2.5317E-06" ixz="-1.6036E-06" iyy="0.00049449" iyz="0.0001344" izz="0.0001125" />
+      <origin
+        xyz="0.029606 -0.056108 0.013102"
+        rpy="-0.175 0 0" />
+      <mass
+        value="0.01" />
+      <inertia
+        ixx="0.00051563"
+        ixy="2.5317E-06"
+        ixz="-1.6036E-06"
+        iyy="0.00049449"
+        iyz="0.0001344"
+        izz="0.0001125" />
     </inertial>
     <visual>
-      <origin xyz="-0.0035 0.02 0.024" rpy="0 0 0" />
-      <geometry>
-        <mesh filename="$(arg mesh_dir)/meshes/foot.dae" />
+      <origin
+        xyz="-0.0035 0.02 0.024"
+        rpy="0 0 0" />
+      <geometry>
+        <mesh
+          filename="$(arg mesh_dir)/meshes/foot.dae" />
       </geometry>
       <material name="">
@@ -263,9 +355,16 @@
         </pbr>
       </material>
+      <!-- <material
+        name="">
+        <color
+          rgba="0.79216 0.81961 0.93333 1" />
+      </material> -->
     </visual>
     <collision>
-      <origin xyz="0.029606 -0.065 0.05" rpy="0 0 0" />
-      <geometry>
-        <box size="0.0675 0.025 0.2" />
+      <origin
+        xyz="0.029606 -0.065 0.05"
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
Commit message: Added loadcell sensor -t /loadcell/osl_foot

File: src/ros2_jazzy/urdf/newoslsim.xacro (robot description, xacro)
@@ -410,5 +410,5 @@
     <limit effort="1.0" velocity="100" lower="-1.57" upper="1.57" />
   </joint>
-<link name="osl_foot">
+  <link name="osl_foot">
     <inertial>
       <origin
@@ -532,9 +532,31 @@
       <mu2>0.5</mu2>
   </gazebo>
-  <joint name="osl_foot_loadcell_link_joint" type="fixed">
-      <parent link="osl_foot"/>
-      <child link="osl_foot_loadcell_link"/>
-      <origin xyz="-0.03 -0.065 0.03" rpy="0 0 0"/>
-  </joint>
+  <gazebo reference="osl_foot_loadcell_link">
+    <kp>1000.0</kp>
+    <kd>1000.0</kd>
+    <mu1>0.5</mu1>
+    <mu2>0.5</mu2>
+    <preserveFixedJoint>true</preserveFixedJoint>  <!-- ADD THIS -->
+  </gazebo>
+  <!-- CHANGE THIS -->
+  <joint name="osl_foot_loadcell_link_joint" type="revolute">
+    <parent link="osl_foot"/>
+    <child link="osl_foot_loadcell_link"/>
+    <origin xyz="-0.03 -0.065 0.03" rpy="0 0 0"/>
+    <axis xyz="1 0 0"/>
+    <limit effort="0" lower="0" upper="0" velocity="0"/>  <!-- zero limits = acts fixed -->
+    <dynamics damping="0.0" friction="0.0"/>
+  </joint>
+  <gazebo reference="osl_foot_loadcell_link_joint">
+    <sensor name="loadcell" type="force_torque">
+      <always_on>true</always_on>
+      <update_rate>100</update_rate>
+      <topic>/loadcell/osl_foot</topic>
+      <force_torque>
+        <frame>child</frame>
+        <measure_direction>child_to_parent</measure_direction>
+      </force_torque>
+    </sensor>
+  </gazebo>
   <gazebo reference="osl_foot_loadcell_link">
     <sensor name='sensor_contact' type='contact'>
@@ -614,4 +636,9 @@
   </gazebo>
   <gazebo>
+    <plugin filename="gz-sim-forcetorque-system"
+            name="gz::sim::systems::ForceTorque">
+    </plugin>
+  </gazebo>
+  <gazebo>
     <plugin filename="gz-sim-touchplugin-system"
           name="gz::sim::systems::TouchPlugin">

Commit message: FIX: updated effort limit to overcome friction force

File: src/ros2_jazzy/urdf/newoslsim.xacro (robot description, xacro)
@@ -141,5 +141,5 @@
     <axis xyz="-0.03 1 0" />
     <dynamics damping="0.5" friction="0.5"/>
-    <limit effort="1.0" velocity="100" lower="-1.57" upper="1.57" />
+    <limit effort="10.0" velocity="100" lower="-1.57" upper="1.57" />
   </joint>
     <link name="socket">
@@ -195,5 +195,5 @@
     <axis xyz="0 1 0" />
     <dynamics damping="0.5" friction="0.5"/>
-    <limit effort="1.0" velocity="100" lower="-1.57" upper="1.57" />
+    <limit effort="10.0" velocity="100" lower="-1.57" upper="1.57" />
   </joint>
   <link name="shin">
@@ -255,5 +255,5 @@
       xyz="0 0 1" />
     <dynamics damping="0.5" friction="0.5"/>
-    <limit effort="1.0" velocity="100" lower="-1.57" upper="1.57" />
+    <limit effort="10.0" velocity="100" lower="-1.57" upper="1.57" />
   </joint>
   <link name="osl_shank">
@@ -323,5 +323,5 @@
       xyz="0 0 1" />
     <dynamics damping="0.5" friction="0.5"/>
-    <limit effort="1.0" velocity="100" lower="-1.57" upper="1.57" />
+    <limit effort="10.0" velocity="100" lower="-1.57" upper="1.57" />
   </joint>
   <link name="foot">
@@ -408,5 +408,5 @@
       xyz="1 0 0" />
     <dynamics damping="0.5" friction="0.5"/>
-    <limit effort="1.0" velocity="100" lower="-1.57" upper="1.57" />
+    <limit effort="10.0" velocity="100" lower="-1.57" upper="1.57" />
   </joint>
   <link name="osl_foot">
@@ -487,5 +487,5 @@
       xyz="0 0 1" />
     <dynamics damping="0.5" friction="0.5"/>
-    <limit effort="1.0" velocity="100" lower="-1.57" upper="1.57" />
+    <limit effort="10.0" velocity="100" lower="-1.57" upper="1.57" />
   </joint>
     <link name="foot_heel">
