Commit message: UPDATE: Hardcoded everything

File: src/ros2_jazzy/urdf/newoslsim.xacro (robot description, xacro)
@@ -297,18 +297,4 @@
     </collision>
   </link>
-  <gazebo reference="osl_shank">
-    <kp>1000.0</kp>
-    <kd>1000.0</kd>
-    <mu1>0.5</mu1>
-    <mu2>0.5</mu2>
-    <!-- Native gz-sim IMU sensor -->
-    <sensor name="osl_foot_imu" type="imu">
-      <always_on>true</always_on>
-      <update_rate>50</update_rate>
-      <visualize>true</visualize>
-      <topic>imu/osl_shank</topic>
-      <pose>0 0 0 0 0 0</pose>
-    </sensor>
-    </gazebo>
 <joint name="osl_knee"
     type="revolute">
@@ -475,4 +461,60 @@
     </collision>
   </link>
+  <link name="imu_shank_link">
+    <inertial>
+      <origin xyz="0 0 0" rpy="0 0 0"/>
+      <mass value="0.00001" />
+      <inertia ixx="1.6e-08" ixy="0.0" ixz="0.0" iyy="1.6e-08" iyz="0.0" izz="1.6e-08"/>
+    </inertial>
+    <collision>
+      <origin xyz="0 0 0" rpy="0 0 0"/>
+      <geometry>
+        <sphere radius="0.020"/>
+      </geometry>
+    </collision>
+  </link>
+  <joint name="imu_shank_link_joint" type="fixed">
+    <parent link="osl_shank"/>
+    <child link="imu_shank_link"/>
+    <origin xyz="0.01 0 0.087" rpy="0 0 0"/>
+  </joint>
+  <gazebo reference="imu_shank_link">
+    <!-- Native gz-sim IMU sensor -->
+    <sensor name="osl_shank_imu" type="imu">
+      <always_on>true</always_on>
+      <update_rate>100</update_rate>
+      <visualize>true</visualize>
+      <topic>imu/osl_shank</topic>
+      <pose>0 0 0 0 0 0</pose>
+    </sensor>
+  </gazebo>
+  <link name="imu_foot_link">
+    <inertial>
+      <origin xyz="0 0 0" rpy="0 0 0"/>
+      <mass value="0.00001" />
+      <inertia ixx="1.6e-08" ixy="0.0" ixz="0.0" iyy="1.6e-08" iyz="0.0" izz="1.6e-08"/>
+    </inertial>
+    <collision>
+      <origin xyz="0 0 0" rpy="0 0 0"/>
+      <geometry>
+        <sphere radius="0.020"/>
+      </geometry>
+    </collision>
+  </link>
+  <joint name="imu_foot_link_joint" type="fixed">
+    <parent link="osl_foot"/>
+    <child link="imu_foot_link"/>
+    <origin xyz="0.01 0 0.05" rpy="0 0 0"/>
+  </joint>
+  <gazebo reference="imu_foot_link">
+    <!-- Native gz-sim IMU sensor -->
+    <sensor name="osl_foot_imu" type="imu">
+      <always_on>true</always_on>
+      <update_rate>100</update_rate>
+      <!-- <visualize>true</visualize> -->
+      <topic>imu/foot</topic>
+      <!-- <pose>0 0 0 0 0 0</pose> -->
+    </sensor>
+  </gazebo>
   <joint name="osl_ankle"
     type="revolute">
@@ -544,7 +586,8 @@
     <child link="osl_foot_loadcell_link"/>
     <origin xyz="-0.03 -0.065 0.03" rpy="0 0 0"/>
-    <axis xyz="1 0 0"/>
-    <limit effort="0" lower="0" upper="0" velocity="0"/>  <!-- zero limits = acts fixed -->
-    <dynamics damping="0.0" friction="0.0"/>
+    <axis
+      xyz="1 0 0" />
+    <dynamics damping="0.5" friction="0.5"/>
+    <limit effort="0.0" velocity="0" lower="0" upper="0" />
   </joint>
   <gazebo reference="osl_foot_loadcell_link_joint">
@@ -578,14 +621,4 @@
     </plugin>
   </gazebo> -->
-  <gazebo reference="osl_foot">
-    <!-- Native gz-sim IMU sensor -->
-    <sensor name="osl_foot_imu" type="imu">
-      <always_on>true</always_on>
-      <update_rate>50</update_rate>
-      <!-- <visualize>true</visualize> -->
-      <topic>imu/foot</topic>
-      <!-- <pose>0 0 0 0 0 0</pose> -->
-    </sensor>
-    </gazebo>
     <ros2_control name="OSLSimSystem" type="system">
       <hardware>
@@ -608,8 +641,8 @@
       </joint>
       <joint name="osl_knee">
-        <command_interface name="effort"/>
+        <command_interface name="position"/>
         <state_interface name="position"/>
         <state_interface name="velocity"/>
-        <state_interface name="effort"/>
+        <!-- <state_interface name="effort"/> -->
       </joint>
       <joint name="ankle">
@@ -619,8 +652,8 @@
       </joint>
       <joint name="osl_ankle">
-        <command_interface name="effort"/>
+        <command_interface name="position"/>
         <state_interface name="position"/>
         <state_interface name="velocity"/>
-        <state_interface name="effort"/>
+        <!-- <state_interface name="effort"/> -->
       </joint>
     </ros2_control>
@@ -666,5 +699,5 @@
       <rpy_offset>0 0 0</rpy_offset>
       <gaussian_noise>0.01</gaussian_noise>
-      <update_rate>50</update_rate>
+      <update_rate>100</update_rate>
     </plugin>
   </gazebo>
