Commit message: motor package

File: install/ros2_jazzy/share/ros2_jazzy/urdf/newoslsim.xacro (robot description, xacro)
@@ -13,4 +13,5 @@
     <parent link="world" />
       <child link="base_link" />
+      <origin xyz="0 0 0.05" rpy="0 0 0"/>
   </joint>
   <link name="slider">

Commit message: motor package

File: install/ros2_jazzy/share/ros2_jazzy/urdf/newoslsim.xacro (robot description, xacro)
@@ -1,11 +1,10 @@
-<?xml version="1.0"?>
-<robot name="oslsim" xmlns:xacro="http://www.ros.org/wiki/xacro">
-    <xacro:arg name="mesh_dir" default="package://ros2_jazzy"/>
-  <link name="world"/>
+<robot xmlns:ns0="http://www.ros.org/wiki/xacro" name="oslsim">
+    <ns0:arg name="mesh_dir" default="package://ros2_jazzy" />
+  <link name="world" />
   <link name="base_link">
     <inertial>
-      <origin rpy="0.0 0 0" xyz="0 0 0"/>
+      <origin rpy="0.0 0 0" xyz="0 0 0" />
       <mass value="0.00001" />
-      <inertia ixx="1.0e-07" ixy="0.0" ixz="0.0" iyy="1.0e-07" iyz="0.0" izz="1.0e-07"/>
+      <inertia ixx="1.0e-07" ixy="0.0" ixz="0.0" iyy="1.0e-07" iyz="0.0" izz="1.0e-07" />
     </inertial>
   </link>
@@ -13,18 +12,16 @@
     <parent link="world" />
       <child link="base_link" />
-      <origin xyz="0 0 0.05" rpy="0 0 0"/>
+      <origin xyz="0 0 0.15" rpy="0 0 0" />
   </joint>
   <link name="slider">
-    <!-- <visual>
-    </visual> -->
-    <inertial>
-        <origin rpy="0.0 0 0" xyz="0 0 0"/>
+    <inertial>
+        <origin rpy="0.0 0 0" xyz="0 0 0" />
         <mass value="0.001" />
-        <inertia ixx="1.0e-07" ixy="0.0" ixz="0.0" iyy="1.0e-07" iyz="0.0" izz="1.0e-07"/>
-    </inertial>
-    <collision>
-        <origin rpy="0.0 0 0" xyz="0 0 0"/>
+        <inertia ixx="1.0e-07" ixy="0.0" ixz="0.0" iyy="1.0e-07" iyz="0.0" izz="1.0e-07" />
+    </inertial>
+    <collision>
+        <origin rpy="0.0 0 0" xyz="0 0 0" />
         <geometry>
-            <box size="0.25 0.25 0.01"/>
+            <box size="0.25 0.25 0.01" />
         </geometry>
     </collision>
@@ -38,16 +35,16 @@
   </gazebo>
   <joint name="slider_joint" type="prismatic">
-      <origin xyz="0 0 0" rpy="0.0 0.0 0.0"/>
+      <origin xyz="0 0 0" rpy="0.0 0.0 0.0" />
       <parent link="base_link" />
       <child link="slider" />
       <axis xyz="1 0 0" />
       <limit effort="1" lower="-10.0" upper="100.0" velocity="1" />
-      <dynamics damping="0.05" friction="0.1"/>
+      <dynamics damping="0.05" friction="0.1" />
   </joint>
   <link name="entity">
       <inertial>
-            <origin rpy="0.0 0 0" xyz="0 0 0"/>
+            <origin rpy="0.0 0 0" xyz="0 0 0" />
             <mass value="0.1" />
-            <inertia ixx="4.16666666667e-05" ixy="0.0" ixz="0.0" iyy="4.16666666667e-05" iyz="0.0" izz="4.16666666667e-05"/>
+            <inertia ixx="4.16666666667e-05" ixy="0.0" ixz="0.0" iyy="4.16666666667e-05" iyz="0.0" izz="4.16666666667e-05" />
         </inertial>
   </link>
@@ -60,22 +57,13 @@
   </gazebo>
   <joint name="entity_joint" type="fixed">
-      <parent link="slider"/>
-      <child link="entity"/>
-      <origin xyz="0 0 -0.05" rpy="0 0 0"/>
+      <parent link="slider" />
+      <child link="entity" />
+      <origin xyz="0 0 -0.05" rpy="0 0 0" />
   </joint>
   <link name="body">
     <inertial>
-      <origin
-        xyz="0 0 0"
-        rpy="0 0 0" />
-      <mass
-        value="0.1" />
-      <inertia
-        ixx="0.001"
-        ixy="0"
-        ixz="0"
-        iyy="0.001"
-        iyz="0"
-        izz="0.001" />
+      <origin xyz="0 0 0" rpy="0 0 0" />
+      <mass value="0.1" />
+      <inertia ixx="0.001" ixy="0" ixz="0" iyy="0.001" iyz="0" izz="0.001" />
     </inertial>
   </link>
@@ -87,44 +75,30 @@
   </gazebo>
   <joint name="root_joint" type="fixed">
-    <parent link="entity"/>
-    <child link="body"/>
+    <parent link="entity" />
+    <child link="body" />
   </joint>
   <link name="thigh">
     <inertial>
-      <origin
-        xyz="0.0079 0.105 -0.18514"
-        rpy="1.5708 0 0" />
-      <mass
-        value="0.55797" />
-      <inertia
-        ixx="0.0451"
-        ixy="-0.0023863"
-        ixz="0.00041503"
-        iyy="0.017843"
-        iyz="-0.00079008"
-        izz="0.046937" />
-    </inertial>
-    <visual>
-      <origin
-        xyz="0 0 -0.004"
-        rpy="0 0 0" />
-      <geometry>
-        <mesh
-          filename="$(arg mesh_dir)/meshes/thigh.dae" />
-      </geometry>
-      <material name="">
-        <pbr>
-          <albedo>0.79216 0.81961 0.93333 1</albedo>
-          <metalness>0.0</metalness>
-          <roughness>0.4</roughness>
-        </pbr>
-      </material>
-    </visual>
-    <collision>
-      <origin
-        xyz="0.0079 0.105 -0.18514"
-        rpy="1.5708 0 0" />
-      <geometry>
-        <box size="0.15 0.3 0.15"/>
+      <origin xyz="0.0079 0.105 -0.18514" rpy="1.5708 0 0" />
+      <mass value="5.0" />
+      <inertia ixx="0.0451" ixy="-0.0023863" ixz="0.00041503" iyy="0.017843" iyz="-0.00079008" izz="0.046937" />
+    </inertial>
+    <visual>
+      <origin xyz="0 0 -0.004" rpy="0 0 0" />
+      <geometry>
+        <mesh filename="$(arg mesh_dir)/meshes/thigh.dae" />
+      </geometry>
+      <material name="">
+        <pbr>
+          <albedo>0.79216 0.81961 0.93333 1</albedo>
+          <metalness>0.0</metalness>
+          <roughness>0.4</roughness>
+        </pbr>
+      </material>
+    </visual>
+    <collision>
+      <origin xyz="0.0079 0.105 -0.18514" rpy="1.5708 0 0" />
+      <geometry>
+        <box size="0.01 0.01 0.01" />
       </geometry>
     </collision>
@@ -137,48 +111,34 @@
   </gazebo>
   <joint name="hip" type="revolute">
-    <parent link="body"/>
-    <child link="thigh"/>
+    <parent link="body" />
+    <child link="thigh" />
     <origin xyz="-0.03 -0.015 0" rpy="0 0 0" />
     <axis xyz="-0.03 1 0" />
-    <dynamics damping="0.5" friction="0.5"/>
+    <dynamics damping="0.5" friction="0.5" />
     <limit effort="1.0" velocity="100" lower="-1.57" upper="1.57" />
   </joint>
     <link name="socket">
     <inertial>
-      <origin
-        xyz="0.0149 -0.105 -0.18907"
-        rpy="1.5708 0 0" />
-      <mass
-        value="0.55993" />
-      <inertia
-        ixx="0.045555"
-        ixy="-0.0028683"
-        ixz="-0.00027507"
-        iyy="0.018107"
-        iyz="0.0020012"
-        izz="0.04735" />
-    </inertial>
-    <visual>
-      <origin
-        xyz="0 0 0"
-        rpy="0 0 0" />
-      <geometry>
-        <mesh
-          filename="$(arg mesh_dir)/meshes/socket.dae" />
-      </geometry>
-      <material name="">
-        <pbr>
-          <albedo>0.79216 0.81961 0.93333 1</albedo>
-          <metalness>0.0</metalness>
-          <roughness>0.4</roughness>
-        </pbr>
-      </material>
-    </visual>
-    <collision>
-      <origin
-        xyz="0.0149 -0.105 -0.18907"
-        rpy="1.5708 0 0" />
-      <geometry>
-        <box size="0.15 0.3 0.15"/>
+      <origin xyz="0.0149 -0.105 -0.18907" rpy="1.5708 0 0" />
+      <mass value="5.0" />
+      <inertia ixx="0.045555" ixy="-0.0028683" ixz="-0.00027507" iyy="0.018107" iyz="0.0020012" izz="0.04735" />
+    </inertial>
+    <visual>
+      <origin xyz="0 0 0" rpy="0 0 0" />
+      <geometry>
+        <mesh filename="$(arg mesh_dir)/meshes/socket.dae" />
+      </geometry>
+      <material name="">
+        <pbr>
+          <albedo>0.79216 0.81961 0.93333 1</albedo>
+          <metalness>0.0</metalness>
+          <roughness>0.4</roughness>
+        </pbr>
+      </material>
+    </visual>
+    <collision>
+      <origin xyz="0.0149 -0.105 -0.18907" rpy="1.5708 0 0" />
+      <geometry>
+        <box size="0.01 0.01 0.01" />
       </geometry>
     </collision>
@@ -191,48 +151,34 @@
   </gazebo>
   <joint name="osl_hip" type="revolute">
-    <parent link="body"/>
-    <child link="socket"/>
+    <parent link="body" />
+    <child link="socket" />
     <origin xyz="0 0.015 0" rpy="0 0 0" />
     <axis xyz="0 1 0" />
-    <dynamics damping="0.5" friction="0.5"/>
+    <dynamics damping="0.5" friction="0.5" />
     <limit effort="1.0" velocity="100" lower="-1.57" upper="1.57" />
   </joint>
   <link name="shin">
     <inertial>
-      <origin
-        xyz="0.00071104 -0.14671 -0.059447"
-        rpy="0 0 0" />
-      <mass
-        value="0.1" />
-      <inertia
-        ixx="0.00092445"
-        ixy="-1.5017E-05"
-        ixz="-2.9597E-06"
-        iyy="0.00064852"
-        iyz="1.2705E-05"
-        izz="0.0013496" />
-    </inertial>
-    <visual>
-      <origin
-        xyz="0.006 0.01 0.006"
-        rpy="0 0 0" />
-      <geometry>
-        <mesh
-          filename="$(arg mesh_dir)/meshes/shin.dae" />
-      </geometry>
-      <material name="">
-        <pbr>
-          <albedo>0.79216 0.81961 0.93333 1</albedo>
-          <metalness>0.0</metalness>
-          <roughness>0.4</roughness>
-        </pbr>
-      </material>
-    </visual>
-    <collision>
-      <origin
-        xyz="0.00071104 -0.14671 -0.059447"
-        rpy="0 0 0" />
-      <geometry>
-        <box size="0.1 0.35 0.1"/>
+      <origin xyz="0.00071104 -0.14671 -0.059447" rpy="0 0 0" />
+      <mass value="3.0" />
+      <inertia ixx="0.00092445" ixy="-1.5017E-05" ixz="-2.9597E-06" iyy="0.00064852" iyz="1.2705E-05" izz="0.0013496" />
+    </inertial>
+    <visual>
+      <origin xyz="0.006 0.01 0.006" rpy="0 0 0" />
+      <geometry>
+        <mesh filename="$(arg mesh_dir)/meshes/shin.dae" />
+      </geometry>
+      <material name="">
+        <pbr>
+          <albedo>0.79216 0.81961 0.93333 1</albedo>
+          <metalness>0.0</metalness>
+          <roughness>0.4</roughness>
+        </pbr>
+      </material>
+    </visual>
+    <collision>
+      <origin xyz="0.00071104 -0.14671 -0.059447" rpy="0 0 0" />
+      <geometry>
+        <box size="0.01 0.01 0.01" />
       </geometry>
     </collision>
@@ -244,55 +190,35 @@
       <mu2>0.5</mu2>
   </gazebo>
-  <joint name="knee"
-    type="revolute">
-    <origin
-      xyz="-0.0073766 0.057865 -0.4427"
-      rpy="1.5708 0 0" />
-    <parent
-      link="thigh" />
-    <child
-      link="shin" />
-    <axis
-      xyz="0 0 1" />
-    <dynamics damping="0.5" friction="0.5"/>
+  <joint name="knee" type="revolute">
+    <origin xyz="-0.0073766 0.057865 -0.4427" rpy="1.5708 0 0" />
+    <parent link="thigh" />
+    <child link="shin" />
+    <axis xyz="0 0 1" />
+    <dynamics damping="0.5" friction="0.5" />
     <limit effort="1.0" velocity="100" lower="-1.57" upper="1.57" />
   </joint>
   <link name="osl_shank">
     <inertial>
-      <origin
-        xyz="0.00071137 -0.14671 0.059447"
-        rpy="0 0 0" />
-      <mass
-        value="0.1" />
-      <inertia
-        ixx="0.00092446"
-        ixy="-1.5017E-05"
-        ixz="2.9586E-06"
-        iyy="0.00064852"
-        iyz="-1.2701E-05"
-        izz="0.0013496" />
-    </inertial>
-    <visual>
-      <origin
-        xyz="0 0 0"
-        rpy="0 0 0" />
-      <geometry>
-        <mesh
-          filename="$(arg mesh_dir)/meshes/osl_shank.dae" />
-      </geometry>
-      <material name="">
-        <pbr>
-          <albedo>0.79216 0.81961 0.93333 1</albedo>
-          <metalness>0.0</metalness>
-          <roughness>0.4</roughness>
-        </pbr>
-      </material>
-    </visual>
-    <collision>
-      <origin
-        xyz="0.00071137 -0.14671 0.059447"
-        rpy="0 0 0" />
-      <geometry>
-        <box size="0.1 0.35 0.1"/>
+      <origin xyz="0.00071137 -0.14671 0.059447" rpy="0 0 0" />
+      <mass value="3.0" />
+      <inertia ixx="0.00092446" ixy="-1.5017E-05" ixz="2.9586E-06" iyy="0.00064852" iyz="-1.2701E-05" izz="0.0013496" />
+    </inertial>
+    <visual>
+      <origin xyz="0 0 0" rpy="0 0 0" />
+      <geometry>
+        <mesh filename="$(arg mesh_dir)/meshes/osl_shank.dae" />
+      </geometry>
+      <material name="">
+        <pbr>
+          <albedo>0.79216 0.81961 0.93333 1</albedo>
+          <metalness>0.0</metalness>
+          <roughness>0.4</roughness>
+        </pbr>
+      </material>
+    </visual>
+    <collision>
+      <origin xyz="0.00071137 -0.14671 0.059447" rpy="0 0 0" />
+      <geometry>
+        <box size="0.01 0.01 0.01" />
       </geometry>
     </collision>
@@ -303,5 +229,4 @@
     <mu1>0.5</mu1>
     <mu2>0.5</mu2>
-    <!-- Native gz-sim IMU sensor -->
     <sensor name="osl_shank_imu" type="imu">
       <always_on>true</always_on>
@@ -312,60 +237,35 @@
     </sensor>
     </gazebo>
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